File: Amp/amp.brd (EAGLE design)
At the start: 97.8 x 53.3 mm, 45 parts, among them IC1 TL072P, Q1 BC550C, Q10 BC560, Q11 IRF520, Q12 IRF520, Q13 IRF520, Q2 BC560, Q3 BC560, Q4 BC550C, Q5 BC560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

Commit message: Oops
Routing:
- net V+: track 189.0 -> 188.1 mm
Changed lines of the file:
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@@
 <wire x1="49.53" y1="17.78" x2="52.705" y2="20.955" width="1.27" layer="16" curve="90"/>
 <wire x1="52.705" y1="20.955" x2="52.705" y2="43.18" width="1.27" layer="16"/>
-<wire x1="50.165" y1="45.72" x2="49.53" y2="45.72" width="1.27" layer="16"/>
 <wire x1="52.705" y1="43.18" x2="67.31" y2="43.18" width="1.27" layer="16"/>
 <wire x1="67.31" y1="43.18" x2="87.63" y2="43.18" width="1.27" layer="16"/>
@@
 <wire x1="40.64" y1="43.18" x2="49.53" y2="43.18" width="1.27" layer="16"/>
 <wire x1="49.53" y1="43.18" x2="52.705" y2="43.18" width="1.27" layer="16"/>
-<wire x1="50.165" y1="45.72" x2="49.53" y2="45.085" width="1.27" layer="16" curve="90"/>
-<wire x1="49.53" y1="45.085" x2="49.53" y2="43.18" width="1.27" layer="16"/>
+<wire x1="49.53" y1="45.72" x2="49.53" y2="43.18" width="1.27" layer="16"/>
 </signal>
 <signal name="V-" class="1">

Commit message: Need to sleep more
Parts:
- added X3: (no value), con-wago-500:W237-102
- moved X2 78.1 mm to (5.08, 36.8), turned to 270 degrees
- moved X1 7.62 mm to (5.08, 19.1)
Connections:
- net GND: now also X3.2
- net IN_L: now also X2.1
- net OUT_L: now also X3.1; no longer X2.1
Routing:
- net IN_L: track 0.00 -> 21.7 mm
- net V-: track 154.1 -> 150.9 mm
Other:
- board text added: "+12"
- board text added: "-12"
- board text added: ">CNAME"
- board text added: ">CREVISION"
- board text added: "Rev:"
Changed lines of the file:
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@@
 <dimension x1="0" y1="53.34" x2="97.79" y2="53.34" x3="48.895" y3="57.15" textsize="1.27" layer="47" dtype="horizontal"/>
 <dimension x1="0" y1="0" x2="0" y2="53.34" x3="-3.81" y3="26.67" textsize="1.27" layer="47" dtype="vertical"/>
+<text x="10.16" y="22.86" size="0.8128" layer="21" ratio="15" rot="R90">+12</text>
+<text x="10.16" y="12.7" size="0.8128" layer="21" ratio="15" rot="R90">-12</text>
+<text x="40.64" y="47.625" size="0.8128" layer="21" ratio="15">&gt;CNAME</text>
+<text x="44.45" y="45.72" size="0.8128" layer="21" ratio="15">&gt;CREVISION</text>
+<text x="40.64" y="45.72" size="0.8128" layer="21" ratio="15">Rev:</text>
 </plain>
 <attributes>
+<attribute name="CNAME" value="Odd Man Out Headphone Amplifier"/>
+<attribute name="CREVISION" value="1"/>
 </attributes>
 <variantdefs>
@@
 <attribute name="VALUE" x="28.194" y="18.796" size="0.8128" layer="27" ratio="15"/>
 </element>
-<element name="X1" library="con-wago-500" package="W237-103" value="" x="5.08" y="26.67" smashed="yes" rot="R270">
-<attribute name="MF" value="" x="5.08" y="26.67" size="1.778" layer="27" rot="R270" display="off"/>
-<attribute name="OC_FARNELL" value="unknown" x="5.08" y="26.67" size="1.778" layer="27" rot="R270" display="off"/>
-<attribute name="OC_NEWARK" value="18M7116" x="5.08" y="26.67" size="1.778" layer="27" rot="R270" display="off"/>
-<attribute name="MPN" value="237-103" x="5.08" y="26.67" size="1.778" layer="27" rot="R270" display="off"/>
-<attribute name="VALUE" x="0.1324" y="31.9748" size="1.27" layer="27" ratio="10" rot="R270"/>
-<attribute name="NAME" x="0.7928" y="27.2758" size="0.8128" layer="25" ratio="15" rot="R270"/>
-</element>
-<element name="X2" library="con-wago-500" package="W237-102" value="" x="82.55" y="26.67" smashed="yes" rot="R90">
+<element name="X1" library="con-wago-500" package="W237-103" value="" x="5.08" y="19.05" smashed="yes" rot="R270">
+<attribute name="MF" value="" x="5.08" y="19.05" size="1.778" layer="27" rot="R270" display="off"/>
+<attribute name="OC_FARNELL" value="unknown" x="5.08" y="19.05" size="1.778" layer="27" rot="R270" display="off"/>
+<attribute name="OC_NEWARK" value="18M7116" x="5.08" y="19.05" size="1.778" layer="27" rot="R270" display="off"/>
+<attribute name="MPN" value="237-103" x="5.08" y="19.05" size="1.778" layer="27" rot="R270" display="off"/>
+<attribute name="VALUE" x="0.1324" y="24.3548" size="1.27" layer="27" ratio="10" rot="R270"/>
+<attribute name="NAME" x="7.1428" y="22.1958" size="0.8128" layer="25" ratio="15" rot="R270"/>
+</element>
+<element name="X3" library="con-wago-500" package="W237-102" value="" x="82.55" y="26.67" smashed="yes" rot="R90">
 <attribute name="MF" value="" x="82.55" y="26.67" size="1.778" layer="27" rot="R90" display="off"/>
 <attribute name="OC_FARNELL" value="unknown" x="82.55" y="26.67" size="1.778" layer="27" rot="R90" display="off"/>
@@
 <attribute name="VALUE" x="90.17" y="21.63" size="1.27" layer="27" ratio="10" rot="R90"/>
 <attribute name="NAME" x="86.9188" y="25.9988" size="0.8128" layer="25" ratio="15" rot="R90"/>
+</element>
+<element name="X2" library="con-wago-500" package="W237-102" value="" x="5.08" y="36.83" smashed="yes" rot="R270">
+<attribute name="MPN" value="237-102" x="5.08" y="36.83" size="1.27" layer="27" rot="R270" display="off"/>
+<attribute name="OC_FARNELL" value="unknown" x="5.08" y="36.83" size="1.27" layer="27" rot="R270" display="off"/>
+<attribute name="OC_NEWARK" value="70K9898" x="5.08" y="36.83" size="1.27" layer="27" rot="R270" display="off"/>
+<attribute name="MF" value="" x="5.08" y="36.83" size="1.27" layer="27" rot="R270" display="off"/>
+<attribute name="VALUE" x="-2.54" y="41.87" size="1.27" layer="27" ratio="10" rot="R270"/>
+<attribute name="NAME" x="7.0612" y="38.1362" size="0.8128" layer="25" ratio="15" rot="R270"/>
 </element>
 </elements>
@@
 <wire x1="13.97" y1="45.72" x2="13.97" y2="40.64" width="1.27" layer="16"/>
 <wire x1="67.31" y1="34.29" x2="73.66" y2="27.94" width="1.27" layer="16" curve="90"/>
-<wire x1="10.16" y1="21.59" x2="10.16" y2="31.75" width="1.27" layer="16"/>
-<wire x1="10.16" y1="31.75" x2="10.16" y2="36.83" width="1.27" layer="16"/>
+<wire x1="10.16" y1="21.59" x2="10.16" y2="24.13" width="1.27" layer="16"/>
+<wire x1="10.16" y1="24.13" x2="10.16" y2="36.83" width="1.27" layer="16"/>
 <wire x1="10.16" y1="36.83" x2="13.97" y2="40.64" width="1.27" layer="16" curve="-90"/>
-<wire x1="3.79" y1="31.67" x2="10.08" y2="31.67" width="1.27" layer="16"/>
-<wire x1="10.08" y1="31.67" x2="10.16" y2="31.75" width="1.27" layer="16" curve="90"/>
 <wire x1="10.16" y1="21.59" x2="13.97" y2="17.78" width="1.27" layer="16" curve="90"/>
 <wire x1="67.31" y1="34.29" x2="67.31" y2="43.18" width="1.27" layer="16"/>
@@
 <wire x1="49.53" y1="43.18" x2="52.705" y2="43.18" width="1.27" layer="16"/>
 <wire x1="49.53" y1="45.72" x2="49.53" y2="43.18" width="1.27" layer="16"/>
+<wire x1="3.79" y1="24.05" x2="10.08" y2="24.05" width="1.27" layer="16"/>
+<wire x1="10.08" y1="24.05" x2="10.16" y2="24.13" width="1.27" layer="16" curve="90"/>
 </signal>
 <signal name="V-" class="1">
@@
 <contactref element="C2" pad="1"/>
 <contactref element="X1" pad="3"/>
-<wire x1="3.79" y1="21.67" x2="12.76" y2="12.7" width="1.27" layer="16" curve="90"/>
-<wire x1="12.76" y1="12.7" x2="44.45" y2="12.7" width="1.27" layer="16"/>
+<wire x1="5.14" y1="12.7" x2="44.45" y2="12.7" width="1.27" layer="16"/>
 <wire x1="44.45" y1="12.7" x2="46.99" y2="12.7" width="1.27" layer="16"/>
 <wire x1="46.99" y1="12.7" x2="58.42" y2="12.7" width="1.27" layer="16"/>
@@
 <wire x1="85.09" y1="10.16" x2="83.82" y2="11.43" width="1.27" layer="16" curve="-90"/>
 <wire x1="83.82" y1="11.43" x2="82.55" y2="12.7" width="1.27" layer="16" curve="90"/>
+<wire x1="5.14" y1="12.7" x2="3.79" y2="14.05" width="1.27" layer="16" curve="-90"/>
 </signal>
 <signal name="N$1">
@@
 <wire x1="17.78" y1="10.16" x2="17.78" y2="15.875" width="0.6096" layer="1"/>
 <wire x1="17.78" y1="15.875" x2="17.78" y2="22.86" width="0.6096" layer="1"/>
-<wire x1="17.78" y1="22.86" x2="17.78" y2="30.48" width="0.6096" layer="16"/>
-<via x="17.78" y="30.48" extent="1-16" drill="0.6"/>
-<wire x1="17.78" y1="30.48" x2="17.78" y2="43.18" width="0.6096" layer="1"/>
+<wire x1="17.78" y1="22.86" x2="17.78" y2="38.1" width="0.6096" layer="16"/>
+<via x="17.78" y="38.1" extent="1-16" drill="0.6"/>
+<wire x1="17.78" y1="38.1" x2="17.78" y2="43.18" width="0.6096" layer="1"/>
 <wire x1="17.78" y1="43.18" x2="20.32" y2="45.72" width="0.6096" layer="1" curve="-90"/>
 <wire x1="36.83" y1="12.7" x2="40.005" y2="15.875" width="0.6096" layer="1" curve="90"/>
@@
 <signal name="IN_L">
 <contactref element="Q1" pad="B"/>
+<contactref element="X2" pad="1"/>
+<wire x1="20.32" y1="30.48" x2="16.51" y2="34.29" width="0.6096" layer="1" curve="-90"/>
+<wire x1="16.51" y1="34.29" x2="16.51" y2="36.83" width="0.6096" layer="1"/>
+<wire x1="16.51" y1="36.83" x2="14.01" y2="39.33" width="0.6096" layer="1" curve="90"/>
+<wire x1="14.01" y1="39.33" x2="3.81" y2="39.33" width="0.6096" layer="1"/>
 </signal>
 <signal name="N$16">
@@
 <contactref element="R21" pad="P$1"/>
 <contactref element="R11" pad="P$2"/>
-<contactref element="X2" pad="1"/>
+<contactref element="X3" pad="1"/>
 <wire x1="38.1" y1="45.72" x2="46.355" y2="37.465" width="0.8128" layer="1" curve="90"/>
 <wire x1="46.355" y1="37.465" x2="80.01" y2="37.465" width="0.8128" layer="1"/>
@@
 </polygon>
 <contactref element="X1" pad="2"/>
-<contactref element="X2" pad="2"/>
+<contactref element="X3" pad="2"/>
 <polygon width="0.4064" layer="16" isolate="0.3048">
 <vertex x="0" y="53.34"/>
@@
 <via x="40.64" y="34.29" extent="1-16" drill="0.6"/>
 <via x="44.45" y="30.48" extent="1-16" drill="0.6"/>
+<contactref element="X2" pad="2"/>
 </signal>
 <signal name="N$26">
