File: Amp/amp.brd (EAGLE design)
At the start: 97.8 x 53.3 mm, 46 parts, among them IC1 TL072P, Q1 BC550C, Q10 BC560, Q11 IRF520, Q12 IRF520, Q13 IRF520, Q2 BC560, Q3 BC560, Q4 BC550C, Q5 BC560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

Commit message: Second channel
Parts:
- removed X3: (no value), con-wago-500:W237-102
- added C10, C8: 1uF, capacitor-wima:C5B5.5
- added C9: 100pF, capacitor-wima:C5B4.5
- added LOGO1: LOGO-MANTIS, my:LOGO-MANTIS
- added Q14, Q17, Q22: BC550C, transistor-npn:TO92-EBC
- added Q15, Q16, Q18, Q19, Q20, Q21, Q23: BC560, transistor-pnp:TO92-EBC
- added Q24, Q25, Q26: IRF520, transistor-power:TO220BV
- added R22, R25: 68, SparkFun-Resistors:AXIAL-0.4
- added R23, R26: 56, SparkFun-Resistors:AXIAL-0.4
- added R24: 11.3, SparkFun-Resistors:AXIAL-0.4
- added R27, R35: 10k, SparkFun-Resistors:AXIAL-0.4
- added R28, R29: 4.99k, SparkFun-Resistors:AXIAL-0.4
- added R30, R33: 33, SparkFun-Resistors:AXIAL-0.4
- added R31, R32: 1Meg, SparkFun-Resistors:AXIAL-0.4
- added R34: 6.81, SparkFun-Resistors:AXIAL-0.4
- added R36: 1.43k, SparkFun-Resistors:AXIAL-0.4
- added R37, R38: 510, SparkFun-Resistors:AXIAL-0.4
- added R39, R40: 100, SparkFun-Resistors:AXIAL-0.4
- added R41, R42: 0.22, SparkFun-Resistors:AXIAL-0.4
- added U4, U6: LM334Z, my:TO-92
- added U5: TL431PTH, SparkFun-AnalogIC:TO-92
- X1: device con-wago-500:W237-103 -> con-wago-508:W237-5P
- X2: device con-wago-500:W237-102 -> con-wago-508:W237-3E
- moved X2 76.3 mm to (81.3, 40.6), turned to 90 degrees
- moved R20 21.9 mm to (80.0, 19.1), turned to 90 degrees
- moved X1 21.7 mm to (2.54, 40.6)
- moved C1 19.1 mm to (29.8, 39.4), turned to 90 degrees
- moved C5 18.0 mm to (40.6, 30.5), turned to 180 degrees
- moved R11 15.4 mm to (36.2, 25.4), turned to 0 degrees
- moved IC1 14.7 mm to (36.2, 40.6), turned to 0 degrees
- moved U1 11.4 mm to (36.8, 16.5)
- moved C3 10.2 mm to (31.8, 30.5), turned to 0 degrees
- moved R10 9.44 mm to (36.2, 21.6), turned to 180 degrees
- moved C2 9.44 mm to (42.5, 39.4)
- moved R3 8.28 mm to (36.2, 12.1), turned to 180 degrees
- moved Q9 8.03 mm to (69.8, 22.9)
- moved Q10 8.03 mm to (69.8, 15.2)
- moved C4 8.03 mm to (53.3, 5.08)
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Connections:
- new net IN_R: Q1.B, X1.5
- new net N$1044: Q26.G, R40.P$1
- new net N$1045: Q23.C, R38.P$1, R40.P$2
- new net N$1046: Q22.E, R37.P$1, R39.P$2
- new net N$1047: Q24.G, R39.P$1
- new net N$27: Q15.B, Q16.B, Q16.C, Q17.C
- new net N$29: Q15.E, R22.P$1
- new net N$30: Q16.E, R25.P$1
- new net N$31: C9.1, Q14.C, Q15.C, Q18.B
- new net N$32: Q14.E, R23.P$2
- new net N$33: Q17.E, R26.P$2
- new net N$34: R23.P$1, R26.P$1, U4.1
- new net N$35: R24.P$2, U4.2
- new net N$36: Q19.B, Q20.B, Q20.C, Q21.E
- new net N$37: Q19.E, R30.P$1
- new net N$38: Q20.E, R33.P$1
- new net N$39: Q18.E, Q19.C, Q21.B
- new net N$40: C9.2, Q21.C, Q22.B, R35.P$2, U5.3
- new net N$41: R35.P$1, R36.P$2, U5.1
- new net N$42: Q23.B, R36.P$1, U5.2, U6.1
- new net N$43: R34.P$2, U6.2
- new net N$48: Q23.E, Q25.S, Q26.D
- new net N$49: Q24.S, R37.P$2, R41.P$1
- new net N$50: Q25.D, Q25.G, R42.P$2
- new net N$51: C8.1, IC1.7, R29.P$1
- new net N$52: C8.2, IC1.6, R31.P$2
- new net N$53: C10.2, IC1.5, R32.P$1
- new net N$54: Q17.B, R27.P$2, R28.P$2, R29.P$2
- new net OUT_R: R11.P$2, R20.P$2, R21.P$1, R6.P$1, X2.1
- net GND: now also C10.1, R28.P$1, R31.P$1, X1.3; no longer X1.2, X3.2
- net IN_L: now also Q14.B, X1.1; no longer Q1.B, X2.1
- net OUT_L: now also R27.P$1, R32.P$2, R41.P$2, R42.P$1, X2.3; no longer R11.P$2, R20.P$2, R21.P$1, R6.P$1, X3.1
- net V+: now also Q22.C, Q24.D, R22.P$2, R25.P$2, R30.P$2, R33.P$2, X1.2; no longer X1.1
- net V-: now also Q18.C, Q26.S, R24.P$1, R34.P$1, R38.P$2, U4.3, U6.3, X1.4; no longer X1.3
Routing:
- net V-: track 150.9 -> 329.2 mm, vias 0 -> 4
- net V+: track 188.1 -> 361.9 mm
- net OUT_R: track 0.00 -> 91.4 mm, vias 0 -> 1
- net N$34: track 0.00 -> 63.7 mm, vias 0 -> 2
- net N$31: track 0.00 -> 61.7 mm, vias 0 -> 1
- net N$40: track 0.00 -> 38.7 mm
- net N$54: track 0.00 -> 37.1 mm
- net N$48: track 0.00 -> 35.0 mm
- net N$49: track 0.00 -> 34.9 mm
- net N$51: track 0.00 -> 31.0 mm
- net N$41: track 0.00 -> 26.8 mm, vias 0 -> 1
- net N$42: track 0.00 -> 24.7 mm
- net N$1044: track 0.00 -> 23.5 mm
- net N$1047: track 0.00 -> 21.4 mm
- net IN_R: track 0.00 -> 19.8 mm, vias 0 -> 2
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Other:
- board size 97.8 x 53.3 mm -> 97.8 x 91.4 mm

Commit message: More gate stoppers
Parts:
- added R43, R44: 100, SparkFun-Resistors:AXIAL-0.4
Connections:
- new net N$44: Q25.G, R43.P$2
- new net N$45: Q12.G, R44.P$2
- net N$25: now also R44.P$1; no longer Q12.G
- net N$50: now also R43.P$1; no longer Q25.G
Routing:
- net N$45: track 0.00 -> 4.86 mm
- net N$44: track 0.00 -> 4.34 mm
- net N$50: track 15.5 -> 19.4 mm
- net N$25: track 12.3 -> 10.5 mm
- net N$23: track 47.3 -> 46.5 mm
- net N$48: track 35.0 -> 34.3 mm
- net N$21: track 34.5 -> 33.7 mm
Changed lines of the file:
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@@
 </element>
 <element name="Q12" library="transistor-power" package="TO220BV" value="IRF520" x="93.98" y="19.05" smashed="yes" rot="R270">
-<attribute name="NAME" x="87.9348" y="24.13" size="0.8128" layer="25" ratio="15" rot="R270"/>
+<attribute name="NAME" x="89.2048" y="26.67" size="0.8128" layer="25" ratio="15" rot="R270"/>
 <attribute name="VALUE" x="86.36" y="24.13" size="0.8128" layer="27" ratio="15" rot="R270"/>
 </element>
@@
 </element>
 <element name="R21" library="SparkFun-Resistors" package="AXIAL-0.4" value="0.22" x="83.82" y="19.05" smashed="yes" rot="R270">
-<attribute name="NAME" x="85.725" y="18.415" size="0.8128" layer="25" font="vector" ratio="15" rot="R270"/>
+<attribute name="NAME" x="81.915" y="17.78" size="0.8128" layer="25" font="vector" ratio="15" rot="R270"/>
 <attribute name="VALUE" x="83.439" y="21.336" size="0.8128" layer="21" font="vector" ratio="15" rot="R270"/>
 </element>
@@
 </element>
 <element name="Q25" library="transistor-power" package="TO220BV" value="IRF520" x="93.98" y="62.23" smashed="yes" rot="R270">
-<attribute name="NAME" x="87.9348" y="67.31" size="0.8128" layer="25" ratio="15" rot="R270"/>
+<attribute name="NAME" x="89.2048" y="69.85" size="0.8128" layer="25" ratio="15" rot="R270"/>
 <attribute name="VALUE" x="86.36" y="67.31" size="0.8128" layer="27" ratio="15" rot="R270"/>
 </element>
@@
 </element>
 <element name="R41" library="SparkFun-Resistors" package="AXIAL-0.4" value="0.22" x="83.82" y="60.96" smashed="yes" rot="R270">
-<attribute name="NAME" x="85.725" y="60.325" size="0.8128" layer="25" font="vector" ratio="15" rot="R270"/>
+<attribute name="NAME" x="81.28" y="59.69" size="0.8128" layer="25" font="vector" ratio="15" rot="R270"/>
 <attribute name="VALUE" x="83.439" y="63.246" size="0.8128" layer="21" font="vector" ratio="15" rot="R270"/>
 </element>
@@
 </element>
 <element name="LOGO1" library="my" package="LOGO-MANTIS" value="LOGO-MANTIS" x="80.01" y="6.35" rot="R90"/>
+<element name="R43" library="SparkFun-Resistors" package="AXIAL-0.4" value="100" x="87.63" y="60.96" smashed="yes" rot="R90">
+<attribute name="NAME" x="86.36" y="57.15" size="0.8128" layer="25" font="vector" ratio="15" rot="R90"/>
+<attribute name="VALUE" x="88.011" y="58.674" size="0.8128" layer="21" font="vector" ratio="15" rot="R90"/>
+</element>
+<element name="R44" library="SparkFun-Resistors" package="AXIAL-0.4" value="100" x="87.63" y="19.05" smashed="yes" rot="R90">
+<attribute name="NAME" x="86.36" y="15.875" size="0.8128" layer="25" font="vector" ratio="15" rot="R90"/>
+<attribute name="VALUE" x="88.011" y="16.764" size="0.8128" layer="21" font="vector" ratio="15" rot="R90"/>
+</element>
 </elements>
 <signals>
@@
 <contactref element="Q13" pad="D"/>
 <contactref element="Q12" pad="S"/>
-<wire x1="91.44" y1="5.08" x2="87.63" y2="8.89" width="0.8128" layer="16" curve="-90"/>
-<wire x1="87.63" y1="8.89" x2="87.63" y2="11.43" width="0.8128" layer="16"/>
-<wire x1="87.63" y1="11.43" x2="87.63" y2="13.97" width="0.8128" layer="16"/>
 <wire x1="74.93" y1="15.24" x2="72.39" y2="17.78" width="0.8128" layer="16" curve="90"/>
 <wire x1="72.39" y1="17.78" x2="71.12" y2="17.78" width="0.8128" layer="16"/>
-<wire x1="87.63" y1="13.97" x2="90.17" y2="16.51" width="0.8128" layer="16" curve="-90"/>
-<wire x1="90.17" y1="16.51" x2="91.44" y2="16.51" width="0.8128" layer="16"/>
 <wire x1="74.93" y1="15.24" x2="78.74" y2="11.43" width="0.8128" layer="16" curve="90"/>
 <wire x1="78.74" y1="11.43" x2="87.63" y2="11.43" width="0.8128" layer="16"/>
+<wire x1="91.44" y1="16.51" x2="91.44" y2="15.24" width="0.8128" layer="16"/>
+<wire x1="91.44" y1="15.24" x2="87.63" y2="11.43" width="0.8128" layer="16" curve="-90"/>
+<wire x1="87.63" y1="11.43" x2="87.63" y2="8.89" width="0.8128" layer="16"/>
+<wire x1="87.63" y1="8.89" x2="91.44" y2="5.08" width="0.8128" layer="16" curve="90"/>
 </signal>
 <signal name="N$23" class="2">
@@
 <contactref element="Q11" pad="S"/>
 <contactref element="R20" pad="P$1"/>
-<wire x1="80.01" y1="13.97" x2="80.01" y2="16.51" width="0.8128" layer="1"/>
-<wire x1="80.01" y1="16.51" x2="85.09" y2="21.59" width="0.8128" layer="1" curve="-90"/>
-<wire x1="85.09" y1="21.59" x2="87.63" y2="24.13" width="0.8128" layer="1" curve="90"/>
-<wire x1="87.63" y1="24.13" x2="87.63" y2="30.48" width="0.8128" layer="1"/>
+<wire x1="80.01" y1="13.97" x2="80.01" y2="17.145" width="0.8128" layer="1"/>
 <via x="78.105" y="30.48" extent="1-16" drill="0.6"/>
 <wire x1="69.85" y1="35.56" x2="67.31" y2="38.1" width="0.8128" layer="1" curve="-90"/>
 <wire x1="78.105" y1="30.48" x2="82.55" y2="30.48" width="0.8128" layer="16"/>
 <via x="82.55" y="30.48" extent="1-16" drill="0.6"/>
-<wire x1="82.55" y1="30.48" x2="87.63" y2="30.48" width="0.8128" layer="1"/>
-<wire x1="87.63" y1="30.48" x2="91.44" y2="30.48" width="0.8128" layer="1"/>
+<wire x1="82.55" y1="30.48" x2="85.725" y2="30.48" width="0.8128" layer="1"/>
+<wire x1="85.725" y1="30.48" x2="91.44" y2="30.48" width="0.8128" layer="1"/>
 <wire x1="78.105" y1="30.48" x2="76.2" y2="32.385" width="0.8128" layer="1" curve="-90"/>
 <wire x1="76.2" y1="32.385" x2="76.2" y2="33.02" width="0.8128" layer="1"/>
 <wire x1="76.2" y1="33.02" x2="73.66" y2="35.56" width="0.8128" layer="1" curve="90"/>
 <wire x1="73.66" y1="35.56" x2="69.85" y2="35.56" width="0.8128" layer="1"/>
+<wire x1="80.01" y1="17.145" x2="82.55" y2="19.685" width="0.8128" layer="1" curve="-90"/>
+<wire x1="82.55" y1="19.685" x2="85.725" y2="22.86" width="0.8128" layer="1" curve="90"/>
+<wire x1="85.725" y1="22.86" x2="85.725" y2="30.48" width="0.8128" layer="1"/>
 </signal>
 <signal name="N$25" class="2">
-<contactref element="Q12" pad="G"/>
 <contactref element="Q12" pad="D"/>
 <contactref element="R21" pad="P$2"/>
-<wire x1="91.44" y1="21.59" x2="91.44" y2="19.05" width="0.8128" layer="1"/>
-<wire x1="83.82" y1="13.97" x2="88.9" y2="19.05" width="0.8128" layer="1" curve="-90"/>
-<wire x1="88.9" y1="19.05" x2="91.44" y2="19.05" width="0.8128" layer="1"/>
+<contactref element="R44" pad="P$1"/>
+<wire x1="91.44" y1="19.05" x2="87.63" y2="15.24" width="0.8128" layer="1" curve="90"/>
+<wire x1="87.63" y1="15.24" x2="87.63" y2="13.97" width="0.8128" layer="1"/>
+<wire x1="87.63" y1="13.97" x2="83.82" y2="13.97" width="0.8128" layer="1"/>
 </signal>
 <signal name="OUT_L" class="2">
@@
 <wire x1="91.44" y1="48.26" x2="87.63" y2="52.07" width="0.8128" layer="16" curve="-90"/>
 <wire x1="87.63" y1="52.07" x2="87.63" y2="53.34" width="0.8128" layer="16"/>
-<wire x1="87.63" y1="53.34" x2="87.63" y2="57.15" width="0.8128" layer="16"/>
 <wire x1="74.93" y1="58.42" x2="72.39" y2="60.96" width="0.8128" layer="16" curve="90"/>
 <wire x1="72.39" y1="60.96" x2="71.12" y2="60.96" width="0.8128" layer="16"/>
-<wire x1="87.63" y1="57.15" x2="90.17" y2="59.69" width="0.8128" layer="16" curve="-90"/>
-<wire x1="90.17" y1="59.69" x2="91.44" y2="59.69" width="0.8128" layer="16"/>
 <wire x1="74.93" y1="58.42" x2="80.01" y2="53.34" width="0.8128" layer="16" curve="90"/>
 <wire x1="80.01" y1="53.34" x2="87.63" y2="53.34" width="0.8128" layer="16"/>
+<wire x1="87.63" y1="53.34" x2="91.44" y2="57.15" width="0.8128" layer="16" curve="90"/>
+<wire x1="91.44" y1="57.15" x2="91.44" y2="59.69" width="0.8128" layer="16"/>
 </signal>
 <signal name="N$49" class="2">
@@
 </signal>
 <signal name="N$50" class="2">
-<contactref element="Q25" pad="G"/>
 <contactref element="Q25" pad="D"/>
 <contactref element="R42" pad="P$2"/>
-<wire x1="91.44" y1="64.77" x2="91.44" y2="62.23" width="0.8128" layer="1"/>
 <wire x1="80.01" y1="66.04" x2="83.82" y2="62.23" width="0.8128" layer="1" curve="90"/>
-<wire x1="83.82" y1="62.23" x2="91.44" y2="62.23" width="0.8128" layer="1"/>
+<wire x1="83.82" y1="62.23" x2="87.63" y2="62.23" width="0.8128" layer="1"/>
+<contactref element="R43" pad="P$1"/>
+<wire x1="87.63" y1="62.23" x2="91.44" y2="62.23" width="0.8128" layer="1"/>
+<wire x1="87.63" y1="55.88" x2="87.63" y2="62.23" width="0.8128" layer="1"/>
 </signal>
 <signal name="N$51">
@@
 <wire x1="78.105" y1="26.67" x2="80.01" y2="26.67" width="0.8128" layer="1"/>
 </signal>
+<signal name="N$44">
+<contactref element="R43" pad="P$2"/>
+<contactref element="Q25" pad="G"/>
+<wire x1="87.63" y1="66.04" x2="88.9" y2="64.77" width="0.8128" layer="1" curve="90"/>
+<wire x1="88.9" y1="64.77" x2="91.44" y2="64.77" width="0.8128" layer="1"/>
+</signal>
+<signal name="N$45">
+<contactref element="R44" pad="P$2"/>
+<contactref element="Q12" pad="G"/>
+<wire x1="87.63" y1="24.13" x2="90.17" y2="21.59" width="0.8128" layer="1" curve="90"/>
+<wire x1="90.17" y1="21.59" x2="91.44" y2="21.59" width="0.8128" layer="1"/>
+</signal>
 </signals>
