File: Amp/amp.sch (EAGLE design)
At the start: 45 parts, among them IC1 TL072P, Q1 BC550C, Q10 BC560, Q11 IRF520, Q12 IRF520, Q13 IRF520, Q2 BC560, Q3 BC560, Q4 BC550C, Q5 BC560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

Commit message: Need to sleep more
Parts:
- added X3: (no value), con-wago-500:W237-102
Connections:
- net GND: now also X3-2.KL
- net IN_L: now also X2-1.KL
- net OUT_L: now also X3-1.KL; no longer X2-1.KL
Other:
- moved on the sheet: X2-1, X2-2
Changed lines of the file:
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@@
 <description>Odd man out headphone amplifier</description>
 <attributes>
-<attribute name="CNAME" value="Odd man out headphone amplifier"/>
+<attribute name="CNAME" value="Odd Man Out Headphone Amplifier"/>
+<attribute name="CREVISION" value="1"/>
 <attribute name="DESIGNER" value="Eugene Zagidullin"/>
 </attributes>
@@
 <part name="GND1" library="SparkFun-Aesthetics" deviceset="GND" device=""/>
 <part name="X1" library="con-wago-500" deviceset="W237-103" device=""/>
+<part name="X3" library="con-wago-500" deviceset="W237-102" device=""/>
+<part name="GND6" library="SparkFun-Aesthetics" deviceset="GND" device=""/>
+<part name="GND8" library="SparkFun-Aesthetics" deviceset="GND" device=""/>
 <part name="X2" library="con-wago-500" deviceset="W237-102" device=""/>
-<part name="GND6" library="SparkFun-Aesthetics" deviceset="GND" device=""/>
 <part name="GND7" library="SparkFun-Aesthetics" deviceset="GND" device=""/>
 </parts>
@@
 <instance part="X1" gate="-2" x="228.6" y="157.48"/>
 <instance part="X1" gate="-3" x="228.6" y="152.4"/>
-<instance part="X2" gate="-1" x="228.6" y="124.46"/>
-<instance part="X2" gate="-2" x="228.6" y="119.38"/>
+<instance part="X3" gate="-1" x="228.6" y="124.46"/>
+<instance part="X3" gate="-2" x="228.6" y="119.38"/>
 <instance part="GND6" gate="1" x="236.22" y="157.48" rot="R90"/>
-<instance part="GND7" gate="1" x="236.22" y="119.38" rot="R90"/>
+<instance part="GND8" gate="1" x="236.22" y="119.38" rot="R90"/>
+<instance part="X2" gate="-1" x="228.6" y="142.24"/>
+<instance part="X2" gate="-2" x="228.6" y="137.16"/>
+<instance part="GND7" gate="1" x="236.22" y="137.16" rot="R90"/>
 </instances>
 <busses>
@@
 <label x="20.32" y="109.22" size="1.778" layer="95" rot="R180" xref="yes"/>
 </segment>
+<segment>
+<pinref part="X2" gate="-1" pin="KL"/>
+<wire x1="233.68" y1="142.24" x2="236.22" y2="142.24" width="0.1524" layer="91"/>
+<label x="236.22" y="142.24" size="1.778" layer="95" xref="yes"/>
+</segment>
 </net>
 <net name="N$16" class="0">
@@
 </segment>
 <segment>
-<pinref part="X2" gate="-1" pin="KL"/>
+<pinref part="X3" gate="-1" pin="KL"/>
 <wire x1="233.68" y1="124.46" x2="236.22" y2="124.46" width="0.1524" layer="91"/>
 <label x="236.22" y="124.46" size="1.778" layer="95" xref="yes"/>
@@
 </segment>
 <segment>
+<pinref part="X3" gate="-2" pin="KL"/>
+<pinref part="GND8" gate="1" pin="GND"/>
+</segment>
+<segment>

Commit message: Second channel
Parts:
- removed X3: (no value), con-wago-500:W237-102
- added C10, C8: 1uF, capacitor-wima:C5/5.5
- added C9: 100pF, capacitor-wima:C5/4.5
- added LOGO1: LOGO-MANTIS, my:LOGO-MANTIS
- added Q14, Q17, Q22: BC550C, transistor-npn:BC550C
- added Q15, Q16, Q18, Q19, Q20, Q21, Q23: BC560, transistor-pnp:BC560
- added Q24, Q25, Q26: IRF520, transistor-power:IRF520
- added R22, R25: 68, SparkFun-Resistors:RESISTORPTH-1/4W
- added R23, R26: 56, SparkFun-Resistors:RESISTORPTH-1/4W
- added R24: 11.3, SparkFun-Resistors:RESISTORPTH-1/4W
- added R27, R35: 10k, SparkFun-Resistors:RESISTORPTH-1/4W
- added R28, R29: 4.99k, SparkFun-Resistors:RESISTORPTH-1/4W
- added R30, R33: 33, SparkFun-Resistors:RESISTORPTH-1/4W
- added R31, R32: 1Meg, SparkFun-Resistors:RESISTORPTH-1/4W
- added R34: 6.81, SparkFun-Resistors:RESISTORPTH-1/4W
- added R36: 1.43k, SparkFun-Resistors:RESISTORPTH-1/4W
- added R37, R38: 510, SparkFun-Resistors:RESISTORPTH-1/4W
- added R39, R40: 100, SparkFun-Resistors:RESISTORPTH-1/4W
- added R41, R42: 0.22, SparkFun-Resistors:RESISTORPTH-1/4W
- added U4, U6: LM334Z, my:LM334Z
- added U5: TL431PTH, SparkFun-AnalogIC:TL431PTH
- X1: device con-wago-500:W237-103 -> con-wago-508:W237-05P
- X2: device con-wago-500:W237-102 -> con-wago-508:W237-3E
Connections:
- new net IN_R: Q1.B, X1-5.KL
- new net N$1044: Q26.G, R40.1
- new net N$1045: Q23.C, R38.1, R40.2
- new net N$1046: Q22.E, R37.1, R39.2
- new net N$1047: Q24.G, R39.1
- new net N$27: Q15.B, Q16.B, Q16.C, Q17.C
- new net N$29: Q15.E, R22.1
- new net N$30: Q16.E, R25.1
- new net N$31: C9.1, Q14.C, Q15.C, Q18.B
- new net N$32: Q14.E, R23.2
- new net N$33: Q17.E, R26.2
- new net N$34: R23.1, R26.1, U4.V+
- new net N$35: R24.2, U4.R
- new net N$36: Q19.B, Q20.B, Q20.C, Q21.E
- new net N$37: Q19.E, R30.1
- new net N$38: Q20.E, R33.1
- new net N$39: Q18.E, Q19.C, Q21.B
- new net N$40: C9.2, Q21.C, Q22.B, R35.2, U5.C
- new net N$41: R35.1, R36.2, U5.R
- new net N$42: Q23.B, R36.1, U5.A, U6.V+
- new net N$43: R34.2, U6.R
- new net N$48: Q23.E, Q25.S, Q26.D
- new net N$49: Q24.S, R37.2, R41.1
- new net N$50: Q25.D, Q25.G, R42.2
- new net N$51: C8.1, IC1B.OUT, R29.1
- new net N$52: C8.2, IC1B.-IN, R31.2
- new net N$53: C10.2, IC1B.+IN, R32.1
- new net N$54: Q17.B, R27.2, R28.2, R29.2
- new net OUT_R: R11.2, R20.2, R21.1, R6.1, X2-1.KL
- net GND: now also C10.1, R28.1, R31.1, X1-3.KL; no longer X1-2.KL, X3-2.KL
- net IN_L: now also Q14.B, X1-1.KL; no longer Q1.B, X2-1.KL
- net OUT_L: now also R27.1, R32.2, R41.2, R42.1, X2-3.KL; no longer R11.2, R20.2, R21.1, R6.1, X3-1.KL
- net V+: now also IC1P.V+, Q22.C, Q24.D, R22.2, R25.2, R30.2, R33.2, X1-2.KL; no longer X1-1.KL
- net V-: now also IC1P.V-, Q18.C, Q26.S, R24.1, R34.1, R38.2, U4.V-, U6.V-, X1-4.KL; no longer X1-3.KL

Commit message: More gate stoppers
Parts:
- added R43, R44: 100, SparkFun-Resistors:RESISTORPTH-1/4W
Connections:
- new net N$44: Q25.G, R43.2
- new net N$45: Q12.G, R44.2
- net N$25: now also R44.1; no longer Q12.G
- net N$50: now also R43.1; no longer Q25.G
Changed lines of the file:
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@@
 <part name="GND3" library="SparkFun-Aesthetics" deviceset="GND" device=""/>
 <part name="LOGO1" library="my" deviceset="LOGO-MANTIS" device=""/>
+<part name="R43" library="SparkFun-Resistors" deviceset="RESISTOR" device="PTH-1/4W" value="100"/>
+<part name="R44" library="SparkFun-Resistors" deviceset="RESISTOR" device="PTH-1/4W" value="100"/>
 </parts>
 <sheets>
@@
 <instance part="GND3" gate="1" x="127" y="-15.24" rot="R90"/>
 <instance part="LOGO1" gate="G$1" x="165.1" y="-15.24"/>
+<instance part="R43" gate="G$1" x="342.9" y="68.58"/>
+<instance part="R44" gate="G$1" x="157.48" y="68.58"/>
 </instances>
 <busses>
@@
 <net name="N$25" class="2">
 <segment>
-<pinref part="Q12" gate="G$1" pin="G"/>
-<wire x1="165.1" y1="68.58" x2="162.56" y2="68.58" width="0.1524" layer="91"/>
-<wire x1="162.56" y1="68.58" x2="162.56" y2="78.74" width="0.1524" layer="91"/>
 <pinref part="Q12" gate="G$1" pin="D"/>
-<wire x1="162.56" y1="78.74" x2="170.18" y2="78.74" width="0.1524" layer="91"/>
 <wire x1="170.18" y1="78.74" x2="170.18" y2="76.2" width="0.1524" layer="91"/>
 <pinref part="R21" gate="G$1" pin="2"/>
 <wire x1="170.18" y1="81.28" x2="170.18" y2="78.74" width="0.1524" layer="91"/>
 <junction x="170.18" y="78.74"/>
+<wire x1="170.18" y1="78.74" x2="149.86" y2="78.74" width="0.1524" layer="91"/>
+<wire x1="149.86" y1="78.74" x2="149.86" y2="68.58" width="0.1524" layer="91"/>
+<pinref part="R44" gate="G$1" pin="1"/>
+<wire x1="149.86" y1="68.58" x2="152.4" y2="68.58" width="0.1524" layer="91"/>
 </segment>
 </net>
@@
 <net name="N$50" class="2">
 <segment>
-<pinref part="Q25" gate="G$1" pin="G"/>
-<wire x1="350.52" y1="68.58" x2="347.98" y2="68.58" width="0.1524" layer="91"/>
-<wire x1="347.98" y1="68.58" x2="347.98" y2="78.74" width="0.1524" layer="91"/>
 <pinref part="Q25" gate="G$1" pin="D"/>
-<wire x1="347.98" y1="78.74" x2="355.6" y2="78.74" width="0.1524" layer="91"/>
 <wire x1="355.6" y1="78.74" x2="355.6" y2="76.2" width="0.1524" layer="91"/>
 <pinref part="R42" gate="G$1" pin="2"/>
 <wire x1="355.6" y1="81.28" x2="355.6" y2="78.74" width="0.1524" layer="91"/>
 <junction x="355.6" y="78.74"/>
+<wire x1="355.6" y1="78.74" x2="335.28" y2="78.74" width="0.1524" layer="91"/>
+<wire x1="335.28" y1="78.74" x2="335.28" y2="68.58" width="0.1524" layer="91"/>
+<pinref part="R43" gate="G$1" pin="1"/>
+<wire x1="335.28" y1="68.58" x2="337.82" y2="68.58" width="0.1524" layer="91"/>
 </segment>
 </net>
@@
 </segment>
 </net>
+<net name="N$44" class="0">
+<segment>
+<pinref part="R43" gate="G$1" pin="2"/>
+<pinref part="Q25" gate="G$1" pin="G"/>
+<wire x1="347.98" y1="68.58" x2="350.52" y2="68.58" width="0.1524" layer="91"/>
+</segment>
+</net>
+<net name="N$45" class="0">
+<segment>
+<pinref part="R44" gate="G$1" pin="2"/>
+<pinref part="Q12" gate="G$1" pin="G"/>
+<wire x1="162.56" y1="68.58" x2="165.1" y2="68.58" width="0.1524" layer="91"/>
+</segment>
+</net>
